File: src/HardwareDesign/RePico.brd (EAGLE design)
At the start: 21 x 51.1 mm, 74 parts, among them IC1 RP2040, IC3 MIC5504-3.3YM5, IC5 MCP6001RT-I/OT, IC8 AP7335-WG-7, J1 JUMPER-3, J2 DNI, J3 JUMPER-3, T1 DMG1012T, X1 12MHz

Commit message: update readme
Parts:
- C23: value 47uF 10V -> 22uF 10V; device ds_capacitors:0805 -> ds_capacitors:0603
- moved C8 10.2 mm to (5.57, 17.5), flipped to the top, turned to 225 degrees
- moved C6 5.34 mm to (11.3, 29.9), flipped to the top, turned to 90 degrees
- moved C10 4.42 mm to (16.4, 25.6), flipped to the top, turned to 0 degrees
- moved C31 3.60 mm to (14.4, 10.2), flipped to the top
- moved C23 1.06 mm to (16.8, 44.8), flipped to the top, turned to 0 degrees
- moved D1 0.52 mm to (17.0, 48.5)
Routing:
- net +3V3: track 117.4 -> 121.3 mm, vias 13 -> 14
- net VCORE_EXT: track 16.7 -> 13.1 mm, vias 4 -> 3
- net V_SYS: track 26.0 -> 23.5 mm
- net GPIO28_ADC_2: track 15.2 -> 16.4 mm
- net GPIO27_ADC1: track 10.2 -> 11.4 mm
- net VREGO: track 21.3 -> 22.2 mm, vias 2 -> 3
- net GPIO29_ADC3: track 25.5 -> 26.4 mm
- net GPIO26_ADC0: track 8.52 -> 9.06 mm
- net GND: track 72.8 -> 72.3 mm, vias 81 -> 82
